File: RASPBERRY_PI_PICO/RP_MODE01.sch (EAGLE design)
At the start: 38 parts, among them U2 RA-02_LORA

Commit message: Se actualiza PCB
Parts:
- added BLUETOOTH: (no value), pinhead:PINHD-1X2
- added PHD_BLUETOOTH: (no value), pinhead:PINHD-1X6
Connections:
- new net ENABLE: PHD_BLUETOOTH.1
- new net RX: BLUETOOTH.1, PHD_BLUETOOTH.5
- new net TX: BLUETOOTH.2, PHD_BLUETOOTH.4
- net GND: now also PHD_BLUETOOTH.3
- net VBUS: now also PHD_BLUETOOTH.2
Changed lines of the file:
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@@
 <part name="S6" library="JS202011SCQN" deviceset="JS202011SCQN" device="" value="SEL3V3"/>
 <part name="JP1" library="pinhead" library_urn="urn:adsk.eagle:library:325" deviceset="PINHD-2X6" device="" package3d_urn="urn:adsk.eagle:package:22474/2"/>
+<part name="PHD_BLUETOOTH" library="pinhead" library_urn="urn:adsk.eagle:library:325" deviceset="PINHD-1X6" device="" package3d_urn="urn:adsk.eagle:package:22472/2"/>
+<part name="BLUETOOTH" library="pinhead" library_urn="urn:adsk.eagle:library:325" deviceset="PINHD-1X2" device="" package3d_urn="urn:adsk.eagle:package:22435/2"/>
 </parts>
 <sheets>
@@
 <attribute name="NAME" x="257.81" y="3.175" size="1.778" layer="95"/>
 <attribute name="VALUE" x="257.81" y="-17.78" size="1.778" layer="96"/>
+</instance>
+<instance part="PHD_BLUETOOTH" gate="A" x="269.24" y="73.66" smashed="yes">
+<attribute name="NAME" x="262.89" y="84.455" size="1.778" layer="95"/>
+<attribute name="VALUE" x="262.89" y="63.5" size="1.778" layer="96"/>
+</instance>
+<instance part="BLUETOOTH" gate="G$1" x="231.14" y="73.66" smashed="yes" rot="R180">
+<attribute name="NAME" x="237.49" y="67.945" size="1.778" layer="95" rot="R180"/>
+<attribute name="VALUE" x="237.49" y="78.74" size="1.778" layer="96" rot="R180"/>
 </instance>
 </instances>
@@
 <wire x1="314.96" y1="55.88" x2="314.96" y2="60.96" width="0.1524" layer="91"/>
 </segment>
+<segment>
+<pinref part="PHD_BLUETOOTH" gate="A" pin="3"/>
+<wire x1="266.7" y1="76.2" x2="238.76" y2="76.2" width="0.1524" layer="91"/>
+<label x="238.76" y="76.2" size="1.778" layer="95"/>
+</segment>
 </net>
 <net name="VBUS" class="0">
@@
 <junction x="314.96" y="71.12"/>
 <label x="314.96" y="73.66" size="1.778" layer="95"/>
+</segment>
+<segment>
+<pinref part="PHD_BLUETOOTH" gate="A" pin="2"/>
+<wire x1="266.7" y1="78.74" x2="238.76" y2="78.74" width="0.1524" layer="91"/>
+<label x="238.76" y="78.74" size="1.778" layer="95"/>
 </segment>
 </net>
@@
 </segment>
 </net>
+<net name="TX" class="0">
+<segment>
+<pinref part="PHD_BLUETOOTH" gate="A" pin="4"/>
+<wire x1="266.7" y1="73.66" x2="233.68" y2="73.66" width="0.1524" layer="91"/>
+<label x="238.76" y="73.66" size="1.778" layer="95"/>
+<pinref part="BLUETOOTH" gate="G$1" pin="2"/>
+</segment>
+</net>
+<net name="RX" class="0">
+<segment>
+<pinref part="PHD_BLUETOOTH" gate="A" pin="5"/>
+<wire x1="266.7" y1="71.12" x2="233.68" y2="71.12" width="0.1524" layer="91"/>
+<label x="238.76" y="71.12" size="1.778" layer="95"/>
+<pinref part="BLUETOOTH" gate="G$1" pin="1"/>
+</segment>
+</net>
+<net name="ENABLE" class="0">
+<segment>
+<pinref part="PHD_BLUETOOTH" gate="A" pin="1"/>
+<wire x1="266.7" y1="81.28" x2="238.76" y2="81.28" width="0.1524" layer="91"/>
+<label x="238.76" y="81.28" size="1.778" layer="95"/>
+</segment>
+</net>
